Commit message: Created  Gazebo

File: description/robot.urdf.xacro (robot description, xacro)
@@ -4,3 +4,4 @@
     <!-- <link name="base_link"></link> -->
     <xacro:include filename="robot_core.xacro" />
+    <xacro:include filename="gazebo_control.xacro" />
 </robot>

File: description/robot_core.xacro (robot description, xacro)
@@ -43,4 +43,7 @@
         </inertial>
     </link>
+    <gazebo reference="chassis">
+        <material>Gazebo/White</material>
+    </gazebo>
     <!-- WHEEL LINK -->
     <joint name="left_wheel_joint" type="continuous">
@@ -68,4 +71,7 @@
         </inertial>
     </link>
+    <gazebo reference="left_wheel">
+        <material>Gazebo/Blue</material>
+    </gazebo>
     <joint name="right_wheel_joint" type="continuous">
         <parent link="base_link" />
@@ -92,4 +98,7 @@
         </inertial>
     </link>
+    <gazebo reference="right_wheel">
+        <material>Gazebo/Blue</material>
+    </gazebo>
     <!-- CASTER WHEEL LINK -->
     <joint name="front_caster_wheel_joint" type="fixed">
@@ -116,4 +125,9 @@
         </inertial>
     </link>
+    <gazebo reference="front_caster_wheel">
+        <material>Gazebo/Black</material>
+        <mu1>0.001</mu1>
+        <mu2>0.001</mu2>
+    </gazebo>
     <joint name="rear_caster_wheel_joint" type="fixed">
         <parent link="chassis" />
@@ -139,3 +153,8 @@
         </inertial>
     </link>
+    <gazebo reference="rear_caster_wheel">
+        <material>Gazebo/Black</material>
+        <mu1>0.001</mu1>
+        <mu2>0.001</mu2>
+    </gazebo>
 </robot>

Commit message: Created  Gazebo Lidar

File: description/robot.urdf.xacro (robot description, xacro)
@@ -5,3 +5,4 @@
     <xacro:include filename="robot_core.xacro" />
     <xacro:include filename="gazebo_control.xacro" />
+    <xacro:include filename="lidar.xacro" />
 </robot>

File: description/robot_core.xacro (robot description, xacro)
@@ -12,4 +12,7 @@
     <material name="black">
         <color rgba="0 0 0 1" />
+    </material>
+    <material name="red">
+        <color rgba="1 0.2 0.2 1" />
     </material>
     <!-- BASE LINK -->
